File: hardware/fpga.sch (KiCad schematic (older format))
At the start: 2 parts, among them U1 ECP5U_45_CABGA256

Commit message: pmods connected and routed
Parts:
- removed D?: D, Diode_SMD:D_0805_2012Metric, symbol Device:D
- added J10: Conn_02x05_Odd_Even, symbol Connector_Generic:Conn_02x05_Odd_Even
- added R3: 10k, Resistor_SMD:R_0805_2012Metric, symbol Device:R
Connections:
- net +3V3: now also U1.P10 (CFG_1), J10.1 (Pin_1), R3.1
- net GND: now also U1.N10 (CFG_0), U1.R10 (CFG_2), J10.3 (Pin_3), J10.5 (Pin_5), J10.7 (Pin_7), J10.9 (Pin_9)
- net +2V5: now reaches U1.G11 (VCCAUX[2]), U1.L7 (VCCAUX[2])
- net p2_1: now reaches U1.A2 (PT4A/+/ULC_GPLL1T_IN)
- net p2_7: now reaches U1.A3 (PT6A/+)
- net p2_8: now reaches U1.A4 (PT6B/-)
- net p2_9: now reaches U1.A5 (PT18A/+)
- net p2_10: now reaches U1.A6 (PT18B/-)
- net clk: now reaches U1.A7 (PT38A/+/PCLKT0_0)
- net p1_1: now reaches U1.A8 (PT38B/-/PCLKC0_0)
- net p2_2: now reaches U1.B4 (PT11B/-)
- net p2_3: now reaches U1.B5 (PT15B/-)
- net p2_4: now reaches U1.B6 (PT31B/-)
- net p1_2: now reaches U1.A10 (PT51B/-)
- net p1_8: now reaches U1.A11 (PT71A/+)
- net p1_3: now reaches U1.A12 (PT71B/-)
- net p1_9: now reaches U1.A13 (PT83A/+)
- net p1_4: now reaches U1.A14 (PT83B/-)
- net p1_10: now reaches U1.A15 (PT85B/-/URC_GPLL1C_IN)
- net p1_7: now reaches U1.A9 (PT51A/+)
- net p5_1: now reaches U1.B16 (PR11A/+/URC_GPLL0T_IN/HS/RDQ17)
- net p5_7: now reaches U1.C15 (PR14B/-/HS/RDQ17)
- net p5_2: now reaches U1.C16 (PR14A/+/HS/RDQ17)
- net p5_8: now reaches U1.D16 (PR17A/+/HS/RDQS17)
- net p5_9: now reaches U1.E15 (PR17B/-/HS/RDQSN17)
- net p5_3: now reaches U1.E16 (PR20D/-/RDQ17)
- net p5_4: now reaches U1.F16 (PR23A/+/HS/RDQ29)
- net p5_10: now reaches U1.G16 (PR29A/+/GR_PCLK2_1/HS/RDQS29)
- net p6_1: now reaches U1.J16 (PR32A/+/PCLKT2_1/HS/RDQ29)
- net p6_7: now reaches U1.K16 (PR32C/+/PCLKT2_0/RDQ29)
- net p6_8: now reaches U1.L15 (PR35B/-/PCLKC3_1/HS/RDQ41)
- net p6_2: now reaches U1.L16 (PR35A/+/PCLKT3_1/HS/RDQ41)
- net p6_3: now reaches U1.M16 (PR35C/+/PCLKT3_0/RDQ41)
- net p6_9: now reaches U1.N16 (PR41A/+/HS/RDQS41)
- net p6_4: now reaches U1.P16 (PR44A/+/HS/RDQ41)
- net p6_10: now reaches U1.R16 (PR44B/-/VREF1_3/HS/RDQ41)
- net p3_9: now reaches U1.L1 (PL35A/+/PCLKT6_1/HS/LDQ41)
- net p3_3: now reaches U1.L2 (PL35B/-/PCLKC6_1/HS/LDQ41)
- net p3_8: now reaches U1.M1 (PL35C/+/PCLKT6_0/LDQ41)
- net p3_2: now reaches U1.N1 (PL41A/+/HS/LDQS41)
- net p3_7: now reaches U1.P1 (PL44A/+/HS/LDQ41)
- net p3_1: now reaches U1.R1 (PL44B/-/VREF1_6/HS/LDQ41)
- net button1: now reaches U1.R2 (PL59C/+/LDQ65)
- net led1: now reaches U1.R3 (PL62B/-/HS/LDQ65)
- net gp16: now reaches U1.R4 (PL62C/+/LDQ65)
- net gp12: now reaches U1.R5 (PL65A/+/HS/LDQS65)
- net button2: now reaches U1.T2 (PL59D/-/LDQ65)
- net led2: now reaches U1.T3 (PL62D/-/LDQ65)
- net gp13: now reaches U1.T4 (PL65B/-/HS/LDQSN65)
- net p4_10: now reaches U1.B1 (PL11A/+/ULC_GPLL0T_IN/HS/LDQ17)
- net p4_9: now reaches U1.C1 (PL14A/+/HS/LDQ17)
- net p4_4: now reaches U1.C2 (PL14B/-/HS/LDQ17)
- net p4_3: now reaches U1.D1 (PL17A/+/HS/LDQS17)
- net p4_2: now reaches U1.E1 (PL20D/-/LDQ17)
- net p4_8: now reaches U1.E2 (PL17B/-/HS/LDQSN17)
- net p4_7: now reaches U1.F1 (PL23A/+/HS/LDQ29)
- net p4_1: now reaches U1.G1 (PL29A/+/GR_PCLK7_1/HS/LDQS29)
- net p3_10: now reaches U1.J1 (PL32A/+/PCLKT7_1/HS/LDQ29)
- net p3_4: now reaches U1.K1 (PL32C/+/PCLKT7_0/LDQ29)
- net sd_io2: now reaches U1.M7 (PB9B/-/D2/IO2)
- net sd_io3: now reaches U1.N7 (PB9A/+/D3/IO3)
- net sd_cs: now reaches U1.N8 (PB15A/+/HOLDN/DI/BUSY/CSSPIN/CEN)
- net sd_clk: now reaches U1.N9 (CCLK/MCLK/SCK)
- net sd_clk: now also R3.2
- net cdone: now reaches U1.P9 (DONE)
- net creset: now reaches U1.R9 (PROGRAMN)
- net creset: now also J10.10 (Pin_10)
- net gp6: now reaches U1.T6 (PB4A/+/D7/IO7)
- net sdi: now reaches U1.T7 (PB11A/+/D1/MISO/IO1)
- net sdo: now reaches U1.T8 (PB11B/-/D0/MOSI/IO0)
- net tdo: now reaches U1.M10 (TDO)
- net tdo: now also J10.6 (Pin_6)
- net tdi: now reaches U1.R11 (TDI)
- net tdi: now also J10.8 (Pin_8)
- net tck: now reaches U1.T10 (TCK)
- net tck: now also J10.4 (Pin_4)
- net tms: now reaches U1.T11 (TMS)
- net tms: now also J10.2 (Pin_2)
- net +1V2 renamed +1V1
- no-connect marks 0 -> 8
Other:
- note added: "jtag arm 10 pin pinout\n"
- moved on the sheet: U1H, U1I

Commit message: routed
Parts:
- added R14, R4, R5, R7, R8: 10k, Resistor_SMD:R_0805_2012Metric, symbol Device:R
- J10: footprint (none) -> Connector_PinHeader_1.27mm:PinHeader_2x05_P1.27mm_Vertical
Connections:
- net +3V3: now also R14.2, R5.2, R8.1; no longer U1.P10 (CFG_1)
- net GND: now also R4.1, R7.1; no longer U1.N10 (CFG_0), U1.R10 (CFG_2)
- net creset: now also R14.1
- net sd_cs: now also R8.2
- net ce1: now reaches U1.T13 (PR65B/-/HS/RDQSN65)
- new net: R7.2, U1.N10 (CFG_0)
- new net: R5.1, U1.P10 (CFG_1)
- new net: R4.2, U1.R10 (CFG_2)
- no-connect marks 8 -> 135
Other:
- note added: "cfg[2:0] = 010. MSPI mode"
