File: hardware/fpga.sch (KiCad schematic (older format))
At the start: 8 parts, among them J10 Conn_02x05_Odd_Even, U1 ECP5U_45_CABGA256

Commit message: changes for design review (see readme)
Parts:
- removed R14, R4, R5, R7, R8: 10k, Resistor_SMD:R_0805_2012Metric, symbol Device:R
- added RN1, RN2: 10k, Resistor_SMD:R_Array_Concave_4x0603, symbol Device:R_Pack04_Split
Connections:
- net +3V3: now also RN1.5 (R4.2), RN1.7 (R2.2), RN2.5 (R4.2), RN2.6 (R3.2), RN2.7 (R2.2), RN2.8 (R1.2); no longer R3.1
- net GND: now also R3.1, RN1.6 (R3.2), RN1.8 (R1.2)
- net creset: now also RN1.4 (R4.1)
- net sd_clk: now also RN2.2 (R2.1); no longer R3.2
- net sd_cs: now also RN2.3 (R3.1)
- net sd_io2: now also RN2.1 (R1.1)
- net sd_io3: now also RN2.4 (R4.1)
- net tck: now also R3.2
- net at U1.N10 (CFG_0): now also RN1.1 (R1.1)
- net at U1.P10 (CFG_1): now also RN1.2 (R2.1)
- net at U1.R10 (CFG_2): now also RN1.3 (R3.1)

Commit message: add serial connection
Connections:
- net gp15: now reaches U1.T14 (PR62D/-/RDQ65)
- net gp14: now reaches U1.T15 (PR59D/-/RDQ65)
- no-connect marks 135 -> 133
Changed lines of the file:
@@
 NoConn ~ 9450 4300
 NoConn ~ 9450 4400
-NoConn ~ 9450 4500
 NoConn ~ 9450 4600
 NoConn ~ 9450 4700
 NoConn ~ 9450 4800
-NoConn ~ 9450 4900
 NoConn ~ 9450 5000
 NoConn ~ 9450 5200
@@
 	1    0    0    -1
 $EndComp
+Text GLabel 9450 4900 0    50   Input ~ 0
+gp15
+Text GLabel 9450 4500 0    50   Input ~ 0
+gp14
 $EndSCHEMATC

Commit message: ready to order
Parts:
- added TP2, TP4, TP7: TestPoint, TestPoint:TestPoint_THTPad_D1.0mm_Drill0.5mm, symbol Connector:TestPoint
- J10: footprint Connector_PinHeader_1.27mm:PinHeader_2x05_P1.27mm_Vertical -> Connector_PinHeader_1.27mm:PinHeader_2x05_P1.27mm_Vertical_SMD
Connections:
- net cfg_0: now reaches RN1.1 (R1.1), U1.N10 (CFG_0)
- net cfg_0: now also TP2.1
- net cfg_1: now reaches RN1.2 (R2.1), U1.P10 (CFG_1)
- net cfg_1: now also TP4.1
- net cfg_2: now reaches RN1.3 (R3.1), U1.R10 (CFG_2)
- net cfg_2: now also TP7.1
Changed lines of the file:
@@
 F 0 "J10" H 13000 8917 50  0000 C CNN
 F 1 "Conn_02x05_Odd_Even" H 13000 8826 50  0000 C CNN
-F 2 "Connector_PinHeader_1.27mm:PinHeader_2x05_P1.27mm_Vertical" H 12950 8500 50  0001 C CNN
+F 2 "Connector_PinHeader_1.27mm:PinHeader_2x05_P1.27mm_Vertical_SMD" H 12950 8500 50  0001 C CNN
 F 3 "~" H 12950 8500 50  0001 C CNN
 	1    12950 8500
@@
 Text GLabel 9450 4500 0    50   Input ~ 0
 gp14
+$Comp
+L Connector:TestPoint TP2
+U 1 1 5F17125F
+P 3900 7100
+F 0 "TP2" H 3958 7172 50  0000 L CNN
+F 1 "TestPoint" H 3958 7127 50  0001 L CNN
+F 2 "TestPoint:TestPoint_THTPad_D1.0mm_Drill0.5mm" H 4100 7100 50  0001 C CNN
+F 3 "~" H 4100 7100 50  0001 C CNN
+	1    3900 7100
+	1    0    0    -1
+$EndComp
+$Comp
+L Connector:TestPoint TP4
+U 1 1 5F173D0F
+P 4050 7100
+F 0 "TP4" H 4108 7172 50  0000 L CNN
+F 1 "TestPoint" H 4108 7127 50  0001 L CNN
+F 2 "TestPoint:TestPoint_THTPad_D1.0mm_Drill0.5mm" H 4250 7100 50  0001 C CNN
+F 3 "~" H 4250 7100 50  0001 C CNN
+	1    4050 7100
+	1    0    0    -1
+$EndComp
+$Comp
+L Connector:TestPoint TP7
+U 1 1 5F1748F6
+P 4200 7100
+F 0 "TP7" H 4258 7172 50  0000 L CNN
+F 1 "TestPoint" H 4258 7127 50  0001 L CNN
+F 2 "TestPoint:TestPoint_THTPad_D1.0mm_Drill0.5mm" H 4400 7100 50  0001 C CNN
+F 3 "~" H 4400 7100 50  0001 C CNN
+	1    4200 7100
+	1    0    0    -1
+$EndComp
+Text Label 5000 8050 2    50   ~ 0
+cfg_1
+Text Label 5000 8150 2    50   ~ 0
+cfg_2
+Text Label 4800 7950 0    50   ~ 0
+cfg_0
+Text Label 3900 7100 3    50   ~ 0
+cfg_0
+Text Label 4050 7100 3    50   ~ 0
+cfg_1
+Text Label 4200 7100 3    50   ~ 0
+cfg_2
 $EndSCHEMATC

Commit message: part numbers and notes on dc/dc voltage dividers
Parts:
- R3: manf# (none) -> RC0805FR-0710KL
- U1: manf# ECP5U_45 -> LFE5U-45F-6BG256C‎
Changed lines of the file:
@@
 F 2 "Package_BGA:BGA-256_14.0x14.0mm_Layout16x16_P0.8mm_Ball0.45mm_Pad0.32mm_NSMD" H 9900 9550 60  0001 R CNN
 F 3 "" H 9900 9350 60  0001 R CNN
-F 4 "ECP5U_45" H 9900 9450 60  0001 R CNN "manf#"
+F 4 "LFE5U-45F-6BG256C‎" H 9900 9450 60  0001 R CNN "manf#"
 	1    9750 9500
 	1    0    0    -1
@@
 F 2 "Package_BGA:BGA-256_14.0x14.0mm_Layout16x16_P0.8mm_Ball0.45mm_Pad0.32mm_NSMD" H 1000 2700 60  0001 R CNN
 F 3 "" H 1000 2500 60  0001 R CNN
-F 4 "ECP5U_45" H 1000 2600 60  0001 R CNN "manf#"
+F 4 "LFE5U-45F-6BG256C‎" H 1000 2600 60  0001 R CNN "manf#"
 	2    850  2650
 	1    0    0    -1
@@
 F 2 "Package_BGA:BGA-256_14.0x14.0mm_Layout16x16_P0.8mm_Ball0.45mm_Pad0.32mm_NSMD" H 3300 2250 60  0001 R CNN
 F 3 "" H 3300 2050 60  0001 R CNN
-F 4 "ECP5U_45" H 3300 2150 60  0001 R CNN "manf#"
+F 4 "LFE5U-45F-6BG256C‎" H 3300 2150 60  0001 R CNN "manf#"
 	3    3150 2200
 	1    0    0    -1
@@
 F 2 "Package_BGA:BGA-256_14.0x14.0mm_Layout16x16_P0.8mm_Ball0.45mm_Pad0.32mm_NSMD" H 6150 2450 60  0001 R CNN
 F 3 "" H 6150 2250 60  0001 R CNN
-F 4 "ECP5U_45" H 6150 2350 60  0001 R CNN "manf#"
+F 4 "LFE5U-45F-6BG256C‎" H 6150 2350 60  0001 R CNN "manf#"
 	4    6000 2400
 	1    0    0    -1
@@
 F 2 "Package_BGA:BGA-256_14.0x14.0mm_Layout16x16_P0.8mm_Ball0.45mm_Pad0.32mm_NSMD" H 9600 2650 60  0001 R CNN
 F 3 "" H 9600 2450 60  0001 R CNN
-F 4 "ECP5U_45" H 9600 2550 60  0001 R CNN "manf#"
+F 4 "LFE5U-45F-6BG256C‎" H 9600 2550 60  0001 R CNN "manf#"
 	5    9450 2600
 	1    0    0    -1
@@
 F 2 "Package_BGA:BGA-256_14.0x14.0mm_Layout16x16_P0.8mm_Ball0.45mm_Pad0.32mm_NSMD" H 13450 2450 60  0001 R CNN
 F 3 "" H 13450 2250 60  0001 R CNN
-F 4 "ECP5U_45" H 13450 2350 60  0001 R CNN "manf#"
+F 4 "LFE5U-45F-6BG256C‎" H 13450 2350 60  0001 R CNN "manf#"
 	6    13300 2400
 	1    0    0    -1
@@
 F 2 "Package_BGA:BGA-256_14.0x14.0mm_Layout16x16_P0.8mm_Ball0.45mm_Pad0.32mm_NSMD" H 1200 7050 60  0001 R CNN
 F 3 "" H 1200 6850 60  0001 R CNN
-F 4 "ECP5U_45" H 1200 6950 60  0001 R CNN "manf#"
+F 4 "LFE5U-45F-6BG256C‎" H 1200 6950 60  0001 R CNN "manf#"
 	7    1050 7000
 	1    0    0    -1
@@
 F 2 "Package_BGA:BGA-256_14.0x14.0mm_Layout16x16_P0.8mm_Ball0.45mm_Pad0.32mm_NSMD" H 13900 8400 60  0001 R CNN
 F 3 "" H 13900 8200 60  0001 R CNN
-F 4 "ECP5U_45" H 13900 8300 60  0001 R CNN "manf#"
+F 4 "LFE5U-45F-6BG256C‎" H 13900 8300 60  0001 R CNN "manf#"
 	9    13750 8350
 	1    0    0    -1
@@
 F 2 "Resistor_SMD:R_0805_2012Metric" V 11930 8450 50  0001 C CNN
 F 3 "~" H 12000 8450 50  0001 C CNN
+F 4 "RC0805FR-0710KL" H 12000 8450 50  0001 C CNN "manf#"
 	1    12000 8450
 	-1   0    0    1
@@
 F 2 "Package_BGA:BGA-256_14.0x14.0mm_Layout16x16_P0.8mm_Ball0.45mm_Pad0.32mm_NSMD" H 5600 7900 60  0001 R CNN
 F 3 "" H 5600 7700 60  0001 R CNN
-F 4 "ECP5U_45" H 5600 7800 60  0001 R CNN "manf#"
+F 4 "LFE5U-45F-6BG256C‎" H 5600 7800 60  0001 R CNN "manf#"
 	8    5450 7850
 	1    0    0    -1

Commit message: neaten FPGA page
Other:
- note added: "Config & SPI"
- note added: "JTAG"
- note added: "PSU"
- moved on the sheet: J10, TP2, TP4, TP7, U1A, U1B, U1C, U1D, U1E, U1F, U1G, U1H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

Commit message: * Add missing qspi to the Pi to be able to program bitstream faster. Done
* used IS25LP016D-JBLE as flash, but
 it has problems with enabling QE for QSPI.
Relace with the model used on icebreaker
This is already done, comment should be removed

* ecp5 SPI clock pin can't be used as an input
 so have to [add a bodge wire](https://github.com/mattvenn/basic-ecp5-pcb/issues/3)
for SPI peripheral comms with Pi.
See the test-spi-clk-in branch for a workaround.
Worked around by connecting this pin to a second FPGA pin

* connected I2C pins are just GPIOs. I have found the Pi's I2C hardware unusable, so always use the slower bitbanged version.
Connected I2C pins to official pins.
Removed pull resistors as this is not needed
Parts:
- U1: symbol Lattice_ECP_FPGA:ECP5U_45_CABGA256 -> basic-ecp5-pcb-rescue:ECP5U_45_CABGA256-Lattice_ECP_FPGA
Connections:
- net sd_clk: now also U1.M5 (PL65C/+/LDQ65)
- no-connect marks 133 -> 132
Changed lines of the file:
@@
 $EndDescr
 $Comp
-L Lattice_ECP_FPGA:ECP5U_45_CABGA256 U1
+L basic-ecp5-pcb-rescue:ECP5U_45_CABGA256-Lattice_ECP_FPGA U1
 U 1 1 5F10BE82
 P 10400 7650
+AR Path="/5F10BE82" Ref="U1"  Part="1"
+AR Path="/5F109712/5F10BE82" Ref="U1"  Part="1"
 F 0 "U1" H 11200 8650 118 0000 L CNN
 F 1 "ECP5U_45_CABGA256" H 10150 6550 60  0000 L CNN
@@
 $EndComp
 $Comp
-L Lattice_ECP_FPGA:ECP5U_45_CABGA256 U1
+L basic-ecp5-pcb-rescue:ECP5U_45_CABGA256-Lattice_ECP_FPGA U1
 U 2 1 5F10DDFC
 P 950 2150
+AR Path="/5F10DDFC" Ref="U1"  Part="2"
+AR Path="/5F109712/5F10DDFC" Ref="U1"  Part="2"
 F 0 "U1" H 1700 3200 118 0000 L CNN
 F 1 "ECP5U_45_CABGA256" H 1450 -450 60  0000 L CNN
@@
 $EndComp
 $Comp
-L Lattice_ECP_FPGA:ECP5U_45_CABGA256 U1
+L basic-ecp5-pcb-rescue:ECP5U_45_CABGA256-Lattice_ECP_FPGA U1
 U 3 1 5F111AF1
 P 3550 2150
+AR Path="/5F111AF1" Ref="U1"  Part="3"
+AR Path="/5F109712/5F111AF1" Ref="U1"  Part="3"
 F 0 "U1" H 4300 3200 118 0000 L CNN
 F 1 "ECP5U_45_CABGA256" H 3900 -1200 60  0000 L CNN
@@
 $EndComp
 $Comp
-L Lattice_ECP_FPGA:ECP5U_45_CABGA256 U1
+L basic-ecp5-pcb-rescue:ECP5U_45_CABGA256-Lattice_ECP_FPGA U1
 U 4 1 5F1149C5
 P 6350 2150
+AR Path="/5F1149C5" Ref="U1"  Part="4"
+AR Path="/5F109712/5F1149C5" Ref="U1"  Part="4"
 F 0 "U1" H 7300 3200 118 0000 L CNN
 F 1 "ECP5U_45_CABGA256" H 6900 -1200 60  0000 L CNN
@@
 $EndComp
 $Comp
-L Lattice_ECP_FPGA:ECP5U_45_CABGA256 U1
+L basic-ecp5-pcb-rescue:ECP5U_45_CABGA256-Lattice_ECP_FPGA U1
 U 5 1 5F1182AD
 P 9850 2100
+AR Path="/5F1182AD" Ref="U1"  Part="5"
+AR Path="/5F109712/5F1182AD" Ref="U1"  Part="5"
 F 0 "U1" H 10700 3100 118 0000 L CNN
 F 1 "ECP5U_45_CABGA256" H 10300 -1250 60  0000 L CNN
@@
 $EndComp
 $Comp
-L Lattice_ECP_FPGA:ECP5U_45_CABGA256 U1
+L basic-ecp5-pcb-rescue:ECP5U_45_CABGA256-Lattice_ECP_FPGA U1
 U 6 1 5F120FEF
 P 13250 2050
+AR Path="/5F120FEF" Ref="U1"  Part="6"
+AR Path="/5F109712/5F120FEF" Ref="U1"  Part="6"
 F 0 "U1" H 14200 3000 118 0000 L CNN
 F 1 "ECP5U_45_CABGA256" H 13750 -1300 60  0000 L CNN
@@
 $EndComp
 $Comp
-L Lattice_ECP_FPGA:ECP5U_45_CABGA256 U1
-U 7 1 5F12C303
-P 1450 7400
-F 0 "U1" H 2300 8450 118 0000 L CNN
-F 1 "ECP5U_45_CABGA256" H 1900 4050 60  0000 L CNN
-F 2 "Package_BGA:BGA-256_14.0x14.0mm_Layout16x16_P0.8mm_Ball0.45mm_Pad0.32mm_NSMD" H 1600 7450 60  0001 R CNN
-F 3 "" H 1600 7250 60  0001 R CNN
-F 4 "LFE5U-45F-6BG256C‎" H 1600 7350 60  0001 R CNN "manf#"
-	7    1450 7400
-	1    0    0    -1
-$EndComp
-$Comp
-L Lattice_ECP_FPGA:ECP5U_45_CABGA256 U1
+L basic-ecp5-pcb-rescue:ECP5U_45_CABGA256-Lattice_ECP_FPGA U1
 U 9 1 5F14250E
 P 14200 7450
+AR Path="/5F14250E" Ref="U1"  Part="9"
+AR Path="/5F109712/5F14250E" Ref="U1"  Part="9"
 F 0 "U1" H 14350 7950 118 0000 L CNN
 F 1 "ECP5U_45_CABGA256" H 14250 6900 60  0000 L CNN
@@
 NoConn ~ 13250 3750
 NoConn ~ 13250 4050
-NoConn ~ 13250 4650
 NoConn ~ 13250 4750
 NoConn ~ 13250 4850
@@
 NoConn ~ 13250 5050
 NoConn ~ 13250 5150
-NoConn ~ 1450 7500
 NoConn ~ 1450 7600
 NoConn ~ 1450 7700
@@
 	6250 7450 6600 7450
 $Comp
-L Lattice_ECP_FPGA:ECP5U_45_CABGA256 U1
+L basic-ecp5-pcb-rescue:ECP5U_45_CABGA256-Lattice_ECP_FPGA U1
 U 8 1 5F1343A1
 P 6600 7450
+AR Path="/5F1343A1" Ref="U1"  Part="8"
+AR Path="/5F109712/5F1343A1" Ref="U1"  Part="8"
 F 0 "U1" H 7550 8200 118 0000 L CNN
 F 1 "ECP5U_45_CABGA256" H 7250 5300 60  0000 L CNN
@@
 Text Notes 4600 6200 0    197  Italic 39
 Config & SPI
+$Comp
+L basic-ecp5-pcb-rescue:ECP5U_45_CABGA256-Lattice_ECP_FPGA U1
+U 7 1 5F12C303
+P 1450 7400
+AR Path="/5F12C303" Ref="U1"  Part="7"
+AR Path="/5F109712/5F12C303" Ref="U1"  Part="7"
+F 0 "U1" H 2300 8450 118 0000 L CNN
+F 1 "ECP5U_45_CABGA256" H 1900 4050 60  0000 L CNN
+F 2 "Package_BGA:BGA-256_14.0x14.0mm_Layout16x16_P0.8mm_Ball0.45mm_Pad0.32mm_NSMD" H 1600 7450 60  0001 R CNN
+F 3 "" H 1600 7250 60  0001 R CNN
+F 4 "LFE5U-45F-6BG256C‎" H 1600 7350 60  0001 R CNN "manf#"
+	7    1450 7400
+	1    0    0    -1
+$EndComp
+NoConn ~ 1450 7500
+Text GLabel 13250 4650 0    50   Input ~ 0
+sd_clk
 $EndSCHEMATC
