File: hardware/basic-ecp5-pcb.kicad_pcb (KiCad board)
At the start: 4 copper layers, 100 x 68 mm, 73 parts, among them J1 Conn_01x02, J10 Conn_02x05_Odd_Even, J2 Conn_02x20_Odd_Even, J3 Conn_02x06_Odd_Even, J4 Conn_02x06_Odd_Even, J5 Conn_02x06_Odd_Even, J6 Conn_02x06_Odd_Even, J7 Conn_02x06_Odd_Even, J8 Conn_02x06_Odd_Even, J9 Conn_02x20_Odd_Even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

Commit message: added input R for dc/dc
Parts:
- added R14: 500k, Resistor_SMD:R_0805_2012Metric, F.Cu at (162.2, 57.4)
- renumbered cf0 to TP2, 1 to TP4, 2 to TP7
Routing:
- net +5V: track 77.6 -> 80.2 mm
- net GND: track 80.3 -> 81.7 mm, vias 50 -> 51

Commit message: oshw logo
Parts:
- added G***: LOGO, libs:oshw-logo-small, B.Cu at (93.4, 66.5)
- added G***: LOGO, libs:oshw-logo-small, F.Cu at (93.4, 66.4)
