File: hardware/basic-ecp5-pcb.sch (KiCad schematic (older format))
At the start: 65 parts, among them J1 Conn_01x02, J2 Conn_02x20_Odd_Even, J3 Conn_02x06_Odd_Even, J4 Conn_02x06_Odd_Even, J5 Conn_02x06_Odd_Even, J6 Conn_02x06_Odd_Even, J7 Conn_02x06_Odd_Even, J8 Conn_02x06_Odd_Even, J9 Conn_02x20_Odd_Even, Q1 Q_NMOS_GSD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

Commit message: updated to use icebreaker flash as it works easily for QE
Parts:
- U2: value IS25LP016D-JBLE -> W25Q128JVSIM; manf# IS25LP016D-JBLE-TR‎ -> W25Q128JVSIM
Other:
- note added: "16Mbyte FLASH supports 0Bh fast read. \nSame model as used in IceBreaker"
- note removed: "16Mb FLASH supports 0Bh fast read"
Changed lines of the file:
@@
 P 2450 7600
 F 0 "U2" H 2700 8150 50  0000 C CNN
-F 1 "IS25LP016D-JBLE" H 2450 8350 50  0000 C CNN
+F 1 "W25Q128JVSIM" H 2450 8350 50  0000 C CNN
 F 2 "Package_SO:SOIC-8_5.23x5.23mm_P1.27mm" H 2450 7600 50  0001 C CNN
-F 3 "http://www.farnell.com/datasheets/2622002.pdf?_ga=2.84155929.1437906943.1577705103-1456622639.1577384340" H 2450 7600 50  0001 C CNN
-F 4 "IS25LP016D-JBLE-TR‎" H 2450 7600 50  0001 C CNN "manf#"
+F 3 "https://www.digikey.es/es/datasheets/winbond-electronics/winbond-electronicsw25q128jvdtr20revc200327201820plus" H 2450 7600 50  0001 C CNN
+F 4 "W25Q128JVSIM" H 2450 7600 50  0001 C CNN "manf#"
 	1    2450 7600
 	1    0    0    -1
@@
 $EndComp
 Text Notes 1850 6700 0    50   ~ 0
-16Mb FLASH supports 0Bh fast read
+16Mbyte FLASH supports 0Bh fast read. \nSame model as used in IceBreaker
 $Comp
 L Mechanical:MountingHole_Pad H1

Commit message: * Add missing qspi to the Pi to be able to program bitstream faster. Done
* used IS25LP016D-JBLE as flash, but
 it has problems with enabling QE for QSPI.
Relace with the model used on icebreaker
This is already done, comment should be removed

* ecp5 SPI clock pin can't be used as an input
 so have to [add a bodge wire](https://github.com/mattvenn/basic-ecp5-pcb/issues/3)
for SPI peripheral comms with Pi.
See the test-spi-clk-in branch for a workaround.
Worked around by connecting this pin to a second FPGA pin

* connected I2C pins are just GPIOs. I have found the Pi's I2C hardware unusable, so always use the slower bitbanged version.
Connected I2C pins to official pins.
Removed pull resistors as this is not needed
Parts:
- removed R1, R2: 4.7k, Resistor_SMD:R_0805_2012Metric, symbol Device:R
- X1: symbol clock:SiT2001B -> basic-ecp5-pcb-rescue:SiT2001B-clock
Connections:
- net gp2 is gone; now on net p3_9: J2.3 (Pin_3), J9.3 (Pin_3)
- net gp24 is gone; now on net sd_io2: J2.18 (Pin_18), J9.18 (Pin_18)
- net gp25 is gone; now on net sd_io3: J2.22 (Pin_22), J9.22 (Pin_22)
- net gp3 is gone; now on net p3_10: J2.5 (Pin_5), J9.5 (Pin_5)
- net p3_10: no longer J2.40 (Pin_40), J9.40 (Pin_40)
- net p3_9: no longer J2.38 (Pin_38), J9.38 (Pin_38)
- new net gp20: J2.38 (Pin_38), J9.38 (Pin_38)
- new net gp21: J2.40 (Pin_40), J9.40 (Pin_40)
Changed lines of the file:
@@
 Connection ~ 13150 1150
 $Comp
-L clock:SiT2001B X1
+L basic-ecp5-pcb-rescue:SiT2001B-clock X1
 U 1 1 5E0EF068
 P 1900 4600
@@
 Text Notes 4500 4350 0    50   ~ 0
 ce0
-Text Label 4200 5300 0    50   ~ 0
-gp20
 Text Label 4200 5400 0    50   ~ 0
-gp21
+gp3
 Text Notes 4500 5350 0    50   ~ 0
 used for i2c
@@
 Text Label 4100 5300 2    50   ~ 0
 p3_9
-$Comp
-L Device:R R1
-U 1 1 5EA3B90B
-P 3950 5150
-F 0 "R1" V 3743 5150 50  0001 C CNN
-F 1 "4.7k" V 3950 5150 50  0000 C CNN
-F 2 "Resistor_SMD:R_0805_2012Metric" V 3880 5150 50  0001 C CNN
-F 3 "~" H 3950 5150 50  0001 C CNN
-F 4 "RC0805FR-0710KL" H 3950 5150 50  0001 C CNN "manf#"
-	1    3950 5150
-	0    -1   -1   0
-$EndComp
-$Comp
-L power:+3.3V #PWR0102
-U 1 1 5EA4133C
-P 3800 5150
-F 0 "#PWR0102" H 3800 5000 50  0001 C CNN
-F 1 "+3.3V" H 3815 5323 50  0000 C CNN
-F 2 "" H 3800 5150 50  0001 C CNN
-F 3 "" H 3800 5150 50  0001 C CNN
-	1    3800 5150
-	0    -1   -1   0
-$EndComp
-Wire Wire Line
-	4100 5300 4150 5300
-Wire Wire Line
-	4100 5400 4150 5400
-Wire Wire Line
-	4100 5150 4150 5150
-Wire Wire Line
-	4150 5150 4150 5300
-Connection ~ 4150 5300
-Wire Wire Line
-	4150 5300 4200 5300
-$Comp
-L Device:R R2
-U 1 1 5EA574EA
-P 3950 5500
-F 0 "R2" V 3743 5500 50  0001 C CNN
-F 1 "4.7k" V 3950 5500 50  0000 C CNN
-F 2 "Resistor_SMD:R_0805_2012Metric" V 3880 5500 50  0001 C CNN
-F 3 "~" H 3950 5500 50  0001 C CNN
-F 4 "RC0805FR-0710KL" H 3950 5500 50  0001 C CNN "manf#"
-	1    3950 5500
-	0    -1   -1   0
-$EndComp
-Wire Wire Line
-	4150 5400 4100 5500
-Connection ~ 4150 5400
-Wire Wire Line
-	4150 5400 4200 5400
-$Comp
-L power:+3.3V #PWR0194
-U 1 1 5EA5BBE3
-P 3800 5500
-F 0 "#PWR0194" H 3800 5350 50  0001 C CNN
-F 1 "+3.3V" H 3815 5673 50  0000 C CNN
-F 2 "" H 3800 5500 50  0001 C CNN
-F 3 "" H 3800 5500 50  0001 C CNN
-	1    3800 5500
-	0    -1   -1   0
-$EndComp
 Wire Wire Line
 	4100 5000 4200 5000
@@
 Text Notes 4350 6400 0    197  Italic 39
 Raspberry Pi Pinning
+Wire Wire Line
+	4100 5300 4200 5300
+Text Label 4200 5300 0    50   ~ 0
+gp2
+Wire Wire Line
+	4100 5400 4200 5400
+Text GLabel 5150 4000 0    50   Input ~ 0
+sd_io2
+Text GLabel 5150 4150 0    50   Input ~ 0
+sd_io3
+Text Label 5300 4000 0    50   ~ 0
+gp24
+Wire Wire Line
+	5150 4000 5300 4000
+Text Label 5300 4150 0    50   ~ 0
+gp25
+Wire Wire Line
+	5150 4150 5300 4150
 $EndSCHEMATC
